Commit message: fixed IRB 6600 205 190 mesh path

File: abb_irb6600_support/urdf/irb6600_205_190.urdf (robot description, URDF)
Before this commit: robot abb, 7 links, 6 joints
Links:
- link base_link: geometry collision mesh filename=package://abb_irb6600_support/meshes/irb6600_205_190/base_l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; visual mesh filename=package://abb_irb6600_support/meshes/irb6600_205_190/base_l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
- link link_1: geometry collision mesh filename=package://abb_irb6600_support/meshes/irb6600_205_190/link_1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; visual mesh filename=package://abb_irb6600_support/meshes/irb6600_205_190/link_1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
- link link_2: geometry collision mesh filename=package://abb_irb6600_support/meshes/irb6600_205_190/link_2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; visual mesh filename=package://abb_irb6600_support/meshes/irb6600_205_190/link_2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
- link link_3: geometry collision mesh filename=package://abb_irb6600_support/meshes/irb6600_205_190/link_3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; visual mesh filename=package://abb_irb6600_support/meshes/irb6600_205_190/link_3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
- link link_4: geometry collision mesh filename=package://abb_irb6600_support/meshes/irb6600_205_190/link_4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; visual mesh filename=package://abb_irb6600_support/meshes/irb6600_205_190/link_4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
- link link_5: geometry collision mesh filename=package://abb_irb6600_support/meshes/irb6600_205_190/link_5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; visual mesh filename=package://abb_irb6600_support/meshes/irb6600_205_190/link_5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
- link link_6: geometry collision mesh filename=package://abb_irb6600_support/meshes/irb6600_205_190/link_6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; visual mesh filename=package://abb_irb6600_support/meshes/irb6600_205_190/link_6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

Commit message: added tool mockups to IRB 6600

File: abb_irb6600_support/urdf/irb6600_205_190.urdf (robot description, URDF)
Before this commit: robot abb_irb6600_support_205_190, 7 links, 6 joints
Links:
- added link tool0
- added link tool_mid; collision box size=0.8 0.8 0.48; visual box size=0.8 0.8 0.48
- link base_link: geometry collision mesh filename=package://abb_irb6600_support/meshes/irb6600_205_190//base_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; visual mesh filename=package://abb_irb6600_support/meshes/irb6600_205_190//base_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
- link link_1: geometry collision mesh filename=package://abb_irb6600_support/meshes/irb6600_205_190//link_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; visual mesh filename=package://abb_irb6600_support/meshes/irb6600_205_190//link_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
- link link_2: geometry collision mesh filename=package://abb_irb6600_support/meshes/irb6600_205_190//link_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; visual mesh filename=package://abb_irb6600_support/meshes/irb6600_205_190//link_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
- link link_3: geometry collision mesh filename=package://abb_irb6600_support/meshes/irb6600_205_190//link_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; visual mesh filename=package://abb_irb6600_support/meshes/irb6600_205_190//link_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
- link link_4: geometry collision mesh filename=package://abb_irb6600_support/meshes/irb6600_205_190//link_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; visual mesh filename=package://abb_irb6600_support/meshes/irb6600_205_190//link_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
- link link_5: geometry collision mesh filename=package://abb_irb6600_support/meshes/irb6600_205_190//link_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; visual mesh filename=package://abb_irb6600_support/meshes/irb6600_205_190//link_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
- link link_6: geometry collision mesh filename=package://abb_irb6600_support/meshes/irb6600_205_190//link_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; visual mesh filename=package://abb_irb6600_support/meshes/irb6600_205_190//link_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
Joints:
- removed joint 1
- removed joint 2
- removed joint 3
- removed joint 4
- removed joint 5
- removed joint 6
- added joint joint_1: type revolute, parent base_link, child link_1, origin xyz=0 0 0.2135 rpy=3.14159 -0 0, axis 0 0 1, limit lower=-3.14159 upper=3.14159 effort=10 velocity=10
- added joint joint_2: type revolute, parent link_1, child link_2, origin xyz=0.3 -0.1385 -0.601 rpy=1.5708 1.55799e-24 8.42367e-56, axis 0 0 1, limit lower=-0.733038 upper=1.48353 effort=10 velocity=10
- added joint joint_3: type revolute, parent link_2, child link_3, origin xyz=-2.05391e-15 -0.7 -0.0435 rpy=1.93349e-15 -1.19007e-14 1.55799e-24, axis 0 0 1, limit lower=-1.22173 upper=1.39626 effort=10 velocity=10
- added joint joint_4: type revolute, parent link_3, child link_4, origin xyz=0.14 -0.28 -0.095 rpy=1.62115e-16 -1.5708 0, axis 0 0 1, limit lower=-3.14159 upper=3.14159 effort=10 velocity=10
- added joint joint_5: type revolute, parent link_4, child link_5, origin xyz=-0.103 1.9984e-15 -0.753 rpy=-3.14159 1.5708 0, axis 0 0 1, limit lower=-2.0944 upper=2.0944 effort=10 velocity=10
- added joint joint_6: type revolute, parent link_5, child link_6, origin xyz=0.163 3.33067e-15 -0.103 rpy=-3.14159 1.5708 0, axis 0 0 1, limit lower=-3.14159 upper=3.14159 effort=10 velocity=10
- added joint link_6-tool0: type fixed, parent link_6, child tool0, origin xyz=0.0 0.0 -0.05 rpy=0 3.14159265359 -0.0
- added joint tool0-tool_mid: type fixed, parent tool0, child tool_mid, origin xyz=0.0 0.0 0.5 rpy=0 0 0
