Commit message: adjusted for workspace analysis

File: abb_irb6730_support/urdf/irb6730_210_310.urdf (robot description, URDF)
Before this commit: robot abb_6730, 7 links, 6 joints
Links:
- added link tool0
- added link tool_mid; collision box size=0.8 0.8 0.48; visual box size=0.8 0.8 0.48
- link irb6730_210kg_310_oc_00_base_cad: geometry collision mesh filename=package://abb_irb6730_support/meshes/irb6730_210kg_310_oc_0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; visual mesh filename=package://abb_irb6730_support/meshes/irb6730_210kg_310_oc_0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
- link irb6730_210kg_310_oc_00_link01_cad: geometry collision mesh filename=package://abb_irb6730_support/meshes/irb6730_210kg_310_oc_0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; visual mesh filename=package://abb_irb6730_support/meshes/irb6730_210kg_310_oc_0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
- link irb6730_210kg_310_oc_00_link02_cad: geometry collision mesh filename=package://abb_irb6730_support/meshes/irb6730_210kg_310_oc_0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; visual mesh filename=package://abb_irb6730_support/meshes/irb6730_210kg_310_oc_0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
- link irb6730_210kg_310_oc_00_link03_cad: geometry collision mesh filename=package://abb_irb6730_support/meshes/irb6730_210kg_310_oc_0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; visual mesh filename=package://abb_irb6730_support/meshes/irb6730_210kg_310_oc_0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
- link irb6730_210kg_310_oc_00_link04_cad: geometry collision mesh filename=package://abb_irb6730_support/meshes/irb6730_210kg_310_oc_0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; visual mesh filename=package://abb_irb6730_support/meshes/irb6730_210kg_310_oc_0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
- link irb6730_210kg_310_oc_00_link05_cad: geometry collision mesh filename=package://abb_irb6730_support/meshes/irb6730_210kg_310_oc_0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; visual mesh filename=package://abb_irb6730_support/meshes/irb6730_210kg_310_oc_0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
- link irb6730_210kg_310_oc_00_link06_cad: geometry collision mesh filename=package://abb_irb6730_support/meshes/irb6730_210kg_310_oc_0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; visual mesh filename=package://abb_irb6730_support/meshes/irb6730_210kg_310_oc_0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
Joints:
- added joint link_6-tool0: type fixed, parent irb6730_210kg_310_oc_00_link06_cad, child tool0, origin xyz=0.0 0.0 -0.05 rpy=0 3.14159265359 -0.0
- added joint tool0-tool_mid: type fixed, parent tool0, child tool_mid, origin xyz=0.0 0.0 0.5 rpy=0 0 0
